File: PCB Projects/AlarmClock - Copy/AlarmClock.sch (KiCad schematic (older format))
At the start: 111 parts, among them CON1 BARREL_JACK, IC1 ATMEGA328P-A, J1 HR911105A, P1 CONN_01X04, P2 CONN_01X04, P3 CONN_01X04, P4 CONN_02X03, P5 CONN_02X07, P6 CONN_01X06, Q3 Q_NPN_EBC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

Commit message: More changes
Parts:
- removed R3: 1.5k, Resistors_SMD:R_1206_HandSoldering, symbol R
Connections:
- net labels added: ADXL345-INT1, ADXL345-INT2, ALARM-PWM, DS3232-INT, ROT-1, ROT-2, ROT-BUTTON, Si1145-INT, TSL2581-INT, W5100-CS, W5100-RESET
- net labels removed: PWM
- wire segments 241 -> 242
Changed lines of the file:
@@
 	1    0    0    -1
 $EndComp
-$Comp
-L R R3
-U 1 1 56FFA0B9
-P 4300 1500
-F 0 "R3" V 4380 1500 50  0000 C CNN
-F 1 "1.5k" V 4300 1500 50  0000 C CNN
-F 2 "Resistors_SMD:R_1206_HandSoldering" V 4230 1500 50  0001 C CNN
-F 3 "" H 4300 1500 50  0000 C CNN
-	1    4300 1500
-	1    0    0    -1
-$EndComp
-Text Label 4050 1650 0    60   ~ 0
-PWM
 NoConn ~ 6150 650
 NoConn ~ 4850 950
@@
 	0    1    1    0
 $EndComp
-Text Label 9550 2600 0    60   ~ 0
-PWM
 $Comp
 L BARREL_JACK CON1
@@
 	1    0    0    -1
 $EndComp
-Text Label 4150 1250 0    60   ~ 0
-D5
 $Comp
 L PCF8574TS/3 U5
@@
 $EndComp
 Text Label 3000 4400 0    60   ~ 0
-D4
+ADXL345-INT1
 Text Label 3000 4300 0    60   ~ 0
-D3
+ADXL345-INT2
 $Comp
 L +3.3V #PWR055
@@
 $EndComp
 Text Label 3650 1800 0    60   ~ 0
-D2
+ROT-2
 Text Label 2050 1800 0    60   ~ 0
-D6
+ROT-1
 $Comp
 L GND #PWR069
@@
 $EndComp
 Text Label 3550 1000 0    60   ~ 0
-D7
+ROT-BUTTON
 $Comp
 L +3.3V #PWR070
@@
 MOSI
 Text Label -10750 7000 0    60   ~ 0
-D10
+W5100-CS
 Text Label -10750 7150 0    60   ~ 0
 SCK
@@
 	6400 5250 7050 5250
 Wire Wire Line
-	4050 1650 4550 1650
-Wire Wire Line
-	4550 1650 4550 1250
-Wire Wire Line
-	4550 1250 4850 1250
-Connection ~ 4300 1650
+	4200 1250 4850 1250
 Wire Wire Line
 	7550 800  7550 1400
@@
 	10350 2400 10350 2300
 Wire Wire Line
-	9750 2600 9550 2600
-Wire Wire Line
-	4300 1350 4300 1250
-Wire Wire Line
-	4300 1250 4150 1250
+	9200 2600 9750 2600
 Wire Wire Line
 	7800 1900 7900 1900
@@
 $EndComp
 Text Label 12250 2750 0    60   ~ 0
-D9
+Si1145-INT
 Wire Wire Line
 	12250 2750 12400 2750
@@
 	13650 4400 13750 4400
 Text Label 13650 4200 0    60   ~ 0
-A0
+TSL2581-INT
 Wire Wire Line
 	13650 4200 13750 4200
@@
 Text Label 1050 11600 0    60   ~ 0
 MISO
+Text Label 3450 11450 0    60   ~ 0
+ADXL345-INT1
+Text Label 3450 11300 0    60   ~ 0
+ADXL345-INT1
+Text Label 3450 11150 0    60   ~ 0
+ROT-2
+Text Label 3450 11000 0    60   ~ 0
+ROT-1
+Text Label 3450 10550 0    60   ~ 0
+ROT-BUTTON
+Text Label 4200 1250 0    60   ~ 0
+DS3232-INT
+Text Label 3450 10400 0    60   ~ 0
+DS3232-INT
+Text Label 3450 10250 0    60   ~ 0
+ALARM-PWM
+Text Label 9200 2600 0    60   ~ 0
+ALARM-PWM
+Text Label 3450 10100 0    60   ~ 0
+Si1145-INT
+Text Label 800  10100 0    60   ~ 0
+TSL2581-INT
+Wire Wire Line
+	800  10100 1350 10100
+Text Label 800  11300 0    60   ~ 0
+W5100-CS
+Wire Wire Line
+	850  10550 1350 10550
+Wire Wire Line
+	800  11300 1350 11300
+Text Label 800  11150 0    60   ~ 0
+W5100-RESET
+Wire Wire Line
+	800  11150 1350 11150
+Text Label -7800 4700 0    60   ~ 0
+W5100-RESET
+Wire Wire Line
+	-7800 4700 -7800 4850
+Connection ~ -7800 4850
 $EndSCHEMATC
