File: PCB Projects/AlarmClock/AlarmClock.sch (KiCad schematic (older format))
At the start: 99 parts, among them CON1 BARREL_JACK, J1 HR911105A, P1 CONN_01X04, P2 CONN_01X04, P3 CONN_01X04, P5 CONN_02X07, Q3 Q_NPN_EBC, U1 TSYS01, U10 W5100, U11 TSL2581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

Commit message: More
Parts:
- removed C24, C25: 12pF, Capacitors_SMD:C_1206_HandSoldering, symbol C_Small
- removed C26, C27, C28, C29, C30, C31, C32, C33, C35, C36, C37, C38: 100nF, Capacitors_SMD:C_1206_HandSoldering, symbol C_Small
- removed D10, D11, D6, D7, D8, D9: Led_Small, LEDs:LED_1206, symbol Led_Small
- removed J1: HR911105A, tm-kicad-lib:HR911105a, symbol HR911105A
- removed R1: 12k, Resistors_SMD:R_1206_HandSoldering, symbol R
- removed R2, R4: 10k, Resistors_SMD:R_1206_HandSoldering, symbol R
- removed R20: 300, Resistors_SMD:R_1206_HandSoldering, symbol R
- removed R21, R22, R23, R24, R25, R26, R27, R28: 1k, Resistors_SMD:R_1206_HandSoldering, symbol R
- removed R6: 1M, Resistors_SMD:R_1206_HandSoldering, symbol R
- removed U10: W5100, AJGFEET:W5100, symbol W5100
- removed Y2: 25MHz, Crystals:HC-18UV, symbol Crystal_Small
- added U?: WIZ820io, AJGFEET:WIZ820io, symbol WIZ820io
Connections:
- net labels removed: +1V8
- wire segments 228 -> 153
- no-connect marks 76 -> 41
