File: PCB Projects/Backpack/Backpack.kicad_pcb (KiCad board)
At the start: 2 copper layers, 53.3 x 50.8 mm, 13 parts, among them P1 CONN_01X04, P2 CONN_01X04, P3 CONN_01X04, P4 CONN_01X04, P5 CONN_01X04, U1 UnoBackpack

Commit message: Tweaks
Connections:
- U1 pad 6: (no net) -> GND
- U1 pad 7: (no net) -> GND

Commit message: More
Parts:
- removed C2: .1uF, Capacitors_SMD:C_1206
- removed P3, P5: CONN_01X04, Pin_Headers:Pin_Header_Straight_1x04
- added P8: CONN_01X08, Pin_Headers:Pin_Header_Straight_1x08, F.Cu at (58.4, 80.0)
- added P9: CONN_01X03, Pin_Headers:Pin_Header_Straight_1x03, F.Cu at (63.5, 76.2)
- moved C3 25.4 mm to (68.6, 64.8)
- moved C4 8.89 mm to (61.0, 81.3)
Connections:
- C4 pad 1: +3V3 -> Net-(C4-Pad1)
- U1 pad 29: (no net) -> /IRQ
Routing:
- net /IRQ: track 0.00 -> 32.1 mm
- net +5V: track 47.3 -> 73.0 mm
- net +3V3: track 116.9 -> 92.3 mm, vias 1 -> 0
- net Net-(C4-Pad1): track 0.00 -> 21.9 mm
- net /SCL: track 69.3 -> 57.9 mm
- net GND: track 23.9 -> 16.1 mm
- net /SDA: track 73.8 -> 66.9 mm, vias 1 -> 0
Other:
- board text added: "Gnd"
- board text added: "Vcc"
