File: PCB Projects/Backpack/Backpack.sch (KiCad schematic (older format))
At the start: 13 parts, among them P1 CONN_01X04, P2 CONN_01X04, P3 CONN_01X04, P4 CONN_01X04, P5 CONN_01X04, U1 UnoBackpack

Commit message: Tweaks
Connections:
- wire segments 31 -> 33
Changed lines of the file:
@@
 LIBS:ajglib
 LIBS:Backpack-cache
-LIBS:ProMiniBackplane-cache
 EELAYER 25 0
 EELAYER END
@@
 Wire Wire Line
 	4700 3950 4900 3950
+$Comp
+L GND #PWR019
+U 1 1 57648C9D
+P 3000 3050
+F 0 "#PWR019" H 3000 2800 50  0001 C CNN
+F 1 "GND" H 3000 2900 50  0000 C CNN
+F 2 "" H 3000 3050 50  0000 C CNN
+F 3 "" H 3000 3050 50  0000 C CNN
+	1    3000 3050
+	1    0    0    -1
+$EndComp
+Wire Wire Line
+	3000 3050 3250 3050
+Wire Wire Line
+	3250 3050 3250 2950
 $EndSCHEMATC

Commit message: More
Parts:
- removed C2: .1uF, Capacitors_SMD:C_1206, symbol C_Small
- removed P3, P5: CONN_01X04, Pin_Headers:Pin_Header_Straight_1x04, symbol CONN_01X04
- added P8: CONN_01X08, Pin_Headers:Pin_Header_Straight_1x08, symbol CONN_01X08
- added P9: CONN_01X03, Pin_Headers:Pin_Header_Straight_1x03, symbol CONN_01X03
Connections:
- net labels added: IRQ
- wire segments 33 -> 38
Changed lines of the file:
@@
 	-1   0    0    1
 $EndComp
-$Comp
-L CONN_01X04 P3
-U 1 1 57561591
-P 6700 3350
-F 0 "P3" H 6700 3600 50  0000 C CNN
-F 1 "CONN_01X04" V 6800 3350 50  0000 C CNN
-F 2 "Pin_Headers:Pin_Header_Straight_1x04" H 6700 3350 50  0001 C CNN
-F 3 "" H 6700 3350 50  0000 C CNN
-	1    6700 3350
-	1    0    0    -1
-$EndComp
-$Comp
-L C_Small C2
-U 1 1 57561598
-P 5950 3300
-F 0 "C2" H 5960 3370 50  0000 L CNN
-F 1 ".1uF" H 5960 3220 50  0000 L CNN
-F 2 "Capacitors_SMD:C_1206" H 5950 3300 50  0001 C CNN
-F 3 "" H 5950 3300 50  0000 C CNN
-	1    5950 3300
-	1    0    0    -1
-$EndComp
-$Comp
-L GND #PWR01
-U 1 1 5756159F
-P 5950 3400
-F 0 "#PWR01" H 5950 3150 50  0001 C CNN
-F 1 "GND" H 5950 3250 50  0000 C CNN
-F 2 "" H 5950 3400 50  0000 C CNN
-F 3 "" H 5950 3400 50  0000 C CNN
-	1    5950 3400
-	1    0    0    -1
-$EndComp
-$Comp
-L GND #PWR02
-U 1 1 575615A5
-P 6100 3400
-F 0 "#PWR02" H 6100 3150 50  0001 C CNN
-F 1 "GND" H 6100 3250 50  0000 C CNN
-F 2 "" H 6100 3400 50  0000 C CNN
-F 3 "" H 6100 3400 50  0000 C CNN
-	1    6100 3400
-	1    0    0    -1
-$EndComp
-Text Label 6350 3400 0    60   ~ 0
-SCL
-Text Label 6350 3500 0    60   ~ 0
-SDA
-Wire Wire Line
-	5950 3200 6500 3200
-Wire Wire Line
-	6500 3300 6100 3300
-Wire Wire Line
-	6100 3300 6100 3400
-Wire Wire Line
-	6500 3500 6350 3500
-Wire Wire Line
-	6500 3400 6350 3400
 Wire Wire Line
 	4700 2400 5450 2400
@@
 $EndComp
 $Comp
-L GND #PWR03
+L GND #PWR01
 U 1 1 57561BFE
 P 5950 4050
-F 0 "#PWR03" H 5950 3800 50  0001 C CNN
+F 0 "#PWR01" H 5950 3800 50  0001 C CNN
 F 1 "GND" H 5950 3900 50  0000 C CNN
 F 2 "" H 5950 4050 50  0000 C CNN
@@
 $EndComp
 $Comp
-L GND #PWR04
+L GND #PWR02
 U 1 1 57561C04
 P 6100 4050
-F 0 "#PWR04" H 6100 3800 50  0001 C CNN
+F 0 "#PWR02" H 6100 3800 50  0001 C CNN
 F 1 "GND" H 6100 3900 50  0000 C CNN
 F 2 "" H 6100 4050 50  0000 C CNN
@@
 Wire Wire Line
 	6500 4050 6350 4050
-$Comp
-L CONN_01X04 P5
-U 1 1 57561D7D
-P 6700 4650
-F 0 "P5" H 6700 4900 50  0000 C CNN
-F 1 "CONN_01X04" V 6800 4650 50  0000 C CNN
-F 2 "Pin_Headers:Pin_Header_Straight_1x04" H 6700 4650 50  0001 C CNN
-F 3 "" H 6700 4650 50  0000 C CNN
-	1    6700 4650
-	1    0    0    -1
-$EndComp
 $Comp
 L C_Small C4
@@
 $EndComp
 $Comp
-L GND #PWR05
+L GND #PWR03
 U 1 1 57561D89
 P 5950 4700
-F 0 "#PWR05" H 5950 4450 50  0001 C CNN
+F 0 "#PWR03" H 5950 4450 50  0001 C CNN
 F 1 "GND" H 5950 4550 50  0000 C CNN
 F 2 "" H 5950 4700 50  0000 C CNN
@@
 $EndComp
 $Comp
-L GND #PWR06
+L GND #PWR04
 U 1 1 57561D8F
 P 6100 4700
-F 0 "#PWR06" H 6100 4450 50  0001 C CNN
+F 0 "#PWR04" H 6100 4450 50  0001 C CNN
 F 1 "GND" H 6100 4550 50  0000 C CNN
 F 2 "" H 6100 4700 50  0000 C CNN
@@
 	1    0    0    -1
 $EndComp
-Text Label 6350 4700 0    60   ~ 0
+Text Label 6450 5000 0    60   ~ 0
 SCL
-Text Label 6350 4800 0    60   ~ 0
+Text Label 6450 5200 0    60   ~ 0
 SDA
 Wire Wire Line
-	5950 4500 6500 4500
-Wire Wire Line
-	6500 4600 6100 4600
+	5950 4500 6650 4500
+Wire Wire Line
+	6100 4600 6650 4600
 Wire Wire Line
 	6100 4600 6100 4700
-Wire Wire Line
-	6500 4800 6350 4800
-Wire Wire Line
-	6500 4700 6350 4700
 $Comp
 L CONN_01X04 P2
@@
 $EndComp
 $Comp
-L GND #PWR07
+L GND #PWR05
 U 1 1 57561F07
 P 5950 2750
-F 0 "#PWR07" H 5950 2500 50  0001 C CNN
+F 0 "#PWR05" H 5950 2500 50  0001 C CNN
 F 1 "GND" H 5950 2600 50  0000 C CNN
 F 2 "" H 5950 2750 50  0000 C CNN
@@
 $EndComp
 $Comp
-L GND #PWR08
+L GND #PWR06
 U 1 1 57561F0D
 P 6100 2750
-F 0 "#PWR08" H 6100 2500 50  0001 C CNN
+F 0 "#PWR06" H 6100 2500 50  0001 C CNN
 F 1 "GND" H 6100 2600 50  0000 C CNN
 F 2 "" H 6100 2750 50  0000 C CNN
@@
 $EndComp
 $Comp
-L GND #PWR09
+L GND #PWR07
 U 1 1 5756202C
 P 5300 5750
-F 0 "#PWR09" H 5300 5500 50  0001 C CNN
+F 0 "#PWR07" H 5300 5500 50  0001 C CNN
 F 1 "GND" H 5300 5600 50  0000 C CNN
 F 2 "" H 5300 5750 50  0000 C CNN
@@
 	5300 5750 5400 5750
 $Comp
-L +5V #PWR010
+L +5V #PWR08
 U 1 1 57562699
 P 5300 5450
-F 0 "#PWR010" H 5300 5300 50  0001 C CNN
+F 0 "#PWR08" H 5300 5300 50  0001 C CNN
 F 1 "+5V" H 5300 5590 50  0000 C CNN
 F 2 "" H 5300 5450 50  0000 C CNN
@@
 $EndComp
 $Comp
-L +3V3 #PWR011
+L +3V3 #PWR09
 U 1 1 57562A84
 P 5050 2000
-F 0 "#PWR011" H 5050 1850 50  0001 C CNN
+F 0 "#PWR09" H 5050 1850 50  0001 C CNN
 F 1 "+3V3" H 5050 2140 50  0000 C CNN
 F 2 "" H 5050 2000 50  0000 C CNN
@@
 $EndComp
 $Comp
-L +3V3 #PWR012
+L +3V3 #PWR010
 U 1 1 57562B42
 P 5950 2550
-F 0 "#PWR012" H 5950 2400 50  0001 C CNN
+F 0 "#PWR010" H 5950 2400 50  0001 C CNN
 F 1 "+3V3" H 5950 2690 50  0000 C CNN
 F 2 "" H 5950 2550 50  0000 C CNN
@@
 $EndComp
 $Comp
-L +3V3 #PWR013
-U 1 1 57562BE9
-P 5950 3200
-F 0 "#PWR013" H 5950 3050 50  0001 C CNN
-F 1 "+3V3" H 5950 3340 50  0000 C CNN
-F 2 "" H 5950 3200 50  0000 C CNN
-F 3 "" H 5950 3200 50  0000 C CNN
-	1    5950 3200
-	1    0    0    -1
-$EndComp
-$Comp
-L +3V3 #PWR014
+L +3V3 #PWR011
 U 1 1 57562CE4
 P 5950 3850
-F 0 "#PWR014" H 5950 3700 50  0001 C CNN
+F 0 "#PWR011" H 5950 3700 50  0001 C CNN
 F 1 "+3V3" H 5950 3990 50  0000 C CNN
 F 2 "" H 5950 3850 50  0000 C CNN
@@
 $EndComp
 $Comp
-L +3V3 #PWR015
+L +3V3 #PWR012
 U 1 1 57562D13
-P 5950 4500
-F 0 "#PWR015" H 5950 4350 50  0001 C CNN
-F 1 "+3V3" H 5950 4640 50  0000 C CNN
-F 2 "" H 5950 4500 50  0000 C CNN
-F 3 "" H 5950 4500 50  0000 C CNN
-	1    5950 4500
-	1    0    0    -1
-$EndComp
-$Comp
-L +5V #PWR016
+P 5650 4500
+F 0 "#PWR012" H 5650 4350 50  0001 C CNN
+F 1 "+3V3" H 5650 4640 50  0000 C CNN
+F 2 "" H 5650 4500 50  0000 C CNN
+F 3 "" H 5650 4500 50  0000 C CNN
+	1    5650 4500
+	1    0    0    -1
+$EndComp
+$Comp
+L +5V #PWR013
 U 1 1 57562E56
 P 3050 2850
-F 0 "#PWR016" H 3050 2700 50  0001 C CNN
+F 0 "#PWR013" H 3050 2700 50  0001 C CNN
 F 1 "+5V" H 3050 2990 50  0000 C CNN
 F 2 "" H 3050 2850 50  0000 C CNN
@@
 	3250 2850 3050 2850
 $Comp
-L +3V3 #PWR017
+L +3V3 #PWR014
 U 1 1 57562F65
 P 3150 2750
-F 0 "#PWR017" H 3150 2600 50  0001 C CNN
+F 0 "#PWR014" H 3150 2600 50  0001 C CNN
 F 1 "+3V3" H 3150 2890 50  0000 C CNN
 F 2 "" H 3150 2750 50  0000 C CNN
@@
 $EndComp
 $Comp
-L GND #PWR018
+L GND #PWR015
 U 1 1 57563341
 P 4950 5650
-F 0 "#PWR018" H 4950 5400 50  0001 C CNN
+F 0 "#PWR015" H 4950 5400 50  0001 C CNN
 F 1 "GND" H 4950 5500 50  0000 C CNN
 F 2 "" H 4950 5650 50  0000 C CNN
@@
 	4700 3950 4900 3950
 $Comp
-L GND #PWR019
+L GND #PWR016
 U 1 1 57648C9D
 P 3000 3050
-F 0 "#PWR019" H 3000 2800 50  0001 C CNN
+F 0 "#PWR016" H 3000 2800 50  0001 C CNN
 F 1 "GND" H 3000 2900 50  0000 C CNN
 F 2 "" H 3000 3050 50  0000 C CNN
@@
 Wire Wire Line
 	3250 3050 3250 2950
+$Comp
+L CONN_01X08 P8
+U 1 1 576E40B5
+P 6850 4850
+F 0 "P8" H 6850 5300 50  0000 C CNN
+F 1 "CONN_01X08" V 6950 4850 50  0000 C CNN
+F 2 "Pin_Headers:Pin_Header_Straight_1x08" H 6850 4850 50  0001 C CNN
+F 3 "" H 6850 4850 50  0000 C CNN
+	1    6850 4850
+	1    0    0    -1
+$EndComp
+Wire Wire Line
+	6650 4600 6650 4700
+Wire Wire Line
+	6650 4800 6400 4800
+Wire Wire Line
+	4700 3850 5200 3850
+Text Label 5000 3850 0    60   ~ 0
+IRQ
+Text Label 6450 4900 0    60   ~ 0
+IRQ
+Wire Wire Line
+	6450 4900 6650 4900
+Wire Wire Line
+	6650 5000 6450 5000
+Wire Wire Line
+	6450 5200 6650 5200
+Wire Wire Line
+	6650 5100 6300 5100
+Wire Wire Line
+	6300 5100 6300 4600
+Connection ~ 6300 4600
+Wire Wire Line
+	6400 4800 6400 4500
+Connection ~ 6400 4500
+$Comp
+L +5V #PWR017
+U 1 1 576E47B3
+P 5450 4500
+F 0 "#PWR017" H 5450 4350 50  0001 C CNN
+F 1 "+5V" H 5450 4640 50  0000 C CNN
+F 2 "" H 5450 4500 50  0000 C CNN
+F 3 "" H 5450 4500 50  0000 C CNN
+	1    5450 4500
+	1    0    0    -1
+$EndComp
+$Comp
+L CONN_01X03 P9
+U 1 1 576E4850
+P 5550 4700
+F 0 "P9" H 5550 4900 50  0000 C CNN
+F 1 "CONN_01X03" V 5650 4700 50  0000 C CNN
+F 2 "Pin_Headers:Pin_Header_Straight_1x03" H 5550 4700 50  0001 C CNN
+F 3 "" H 5550 4700 50  0000 C CNN
+	1    5550 4700
+	0    1    1    0
+$EndComp
+Wire Wire Line
+	5950 4500 5950 4300
+Wire Wire Line
+	5950 4300 5550 4300
+Wire Wire Line
+	5550 4300 5550 4500
 $EndSCHEMATC
